File: Hardware/SparkFun_MIDI_Shield.sch (EAGLE design)
At the start: 32 parts, among them J1 MIDI IN, J2 MIDI OUT, J3 UNO_R3_SHIELD, U2 74AHC1G125

Commit message: Updates after engineering review.
Added jumper to allow optional soft serial.
Parts:
- added SJ1: TX sel, SparkFun-Passives:JUMPER-PAD-3-2OF3_NC_BY_TRACE_SMALL
- added SJ2: RX sel, SparkFun-Passives:JUMPER-PAD-3-2OF3_NC_BY_TRACE_SMALL
Connections:
- removed net RX: R2.1, S2.O, U$1.VOUT
- removed net TX: J3.TX, U2.A
- new net HARD-RX: S2.O, SJ1.3
- new net HARD-TX: J3.TX, SJ2.3
- new net PORT-RX: R2.1, SJ1.2, U$1.VOUT
- new net PORT-TX: SJ2.2, U2.A
- new net SOFT-RX: J3.D8, SJ1.1
- new net SOFT-TX: J3.*D9, SJ2.1
Other:
- note added: "MIDI I/O reference design from: http://www.midi.org/techspecs/electrispec.php JP1, JP2, JP3, JP4 implement power-over-MIDI, using pin assignment proposed by Craig Anderton (Pin 1 = Vcc, pin 3 = ground). Close JP1 & 2 to power the MIDI input. Close JP3 & 4 to power the output."
- note added: "SJ1, SJ2 select between hardware serial port (pins 0, 1) and soft-serial (pins 8, 9). Hardware serial selected by default."
- note added: "Serial Port Selection"
- note removed: "MIDI I/O reference design from: http://www.midi.org/techspecs/electrispec.php JP1, JP2, JP3, JP4 implement power-over-MIDI, using pin assignment proposed by Craig Anderton (Pin 1 = Vcc, pin 3 = ground). Close JP1 & 2 to receive power over the MIDI input. Close JP3 & 4 to send power on the output."
- moved on the sheet: J2, JP3, JP4, LED1, LED2, R3, R4, R5, R6, S3, S4, U2

Commit message: Updates after QC checklist.
Parts:
- renumbered U$1 to U1
Other:
- note added: "Shield Vcc is provided by Arduino 5V line. The MIDI standard specifies 5V operation."
Changed lines of the file:
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@@
 <part name="S1" library="SparkFun-Electromechanical" deviceset="SWITCH-MOMENTARY-2" device="SMD" value="Reset"/>
 <part name="S2" library="SparkFun-Electromechanical" deviceset="SWITCH-SPDT" device="SMD" value="RUN/PROGRAM"/>
-<part name="U$1" library="SparkFun-DiscreteSemi" deviceset="OPTO_DARL_6N138S" device="" value="6N138M"/>
 <part name="JP3" library="SparkFun-Passives" deviceset="JUMPER-PAD-2-NO" device="YES_SILK"/>
 <part name="JP4" library="SparkFun-Passives" deviceset="JUMPER-PAD-2-NO" device="YES_SILK"/>
@@
 <part name="SJ1" library="SparkFun-Passives" deviceset="JUMPER-PAD-3-2OF3_NC_BY_TRACE" device="_SMALL" value="TX sel"/>
 <part name="SJ2" library="SparkFun-Passives" deviceset="JUMPER-PAD-3-2OF3_NC_BY_TRACE" device="_SMALL" value="RX sel"/>
+<part name="U1" library="SparkFun-DiscreteSemi" deviceset="OPTO_DARL_6N138S" device="" value="6N138M"/>
 </parts>
 <sheets>
 <sheet>
 <plain>
-<text x="2.54" y="180.594" size="2.54" layer="94">MIDI IN</text>
-<text x="2.54" y="99.06" size="2.54" layer="94">MIDI OUT</text>
+<text x="2.54" y="180.594" size="2.54" layer="97">MIDI IN</text>
+<text x="2.54" y="99.06" size="2.54" layer="97">MIDI OUT</text>
 <text x="172.72" y="7.62" size="2.54" layer="94">Byron Jacquot</text>
 <text x="238.76" y="7.62" size="2.54" layer="94">V1.5</text>
 <wire x1="129.54" y1="185.42" x2="121.92" y2="185.42" width="0.3048" layer="94" style="shortdash"/>
-<wire x1="121.92" y1="185.42" x2="121.92" y2="104.14" width="0.3048" layer="94" style="shortdash"/>
-<wire x1="121.92" y1="104.14" x2="121.92" y2="30.48" width="0.3048" layer="94" style="shortdash"/>
-<wire x1="121.92" y1="30.48" x2="121.92" y2="0" width="0.3048" layer="94" style="shortdash"/>
-<wire x1="0" y1="104.14" x2="86.36" y2="104.14" width="0.3048" layer="94" style="shortdash"/>
-<text x="127" y="180.34" size="2.54" layer="94">Shield Connections and controls</text>
-<wire x1="86.36" y1="104.14" x2="121.92" y2="104.14" width="0.3048" layer="94" style="shortdash"/>
-<wire x1="0" y1="30.48" x2="86.36" y2="30.48" width="0.3048" layer="94" style="shortdash"/>
-<text x="2.54" y="25.4" size="1.778" layer="94" align="top-left">MIDI I/O reference design from:
+<wire x1="121.92" y1="185.42" x2="121.92" y2="104.14" width="0.3048" layer="97" style="shortdash"/>
+<wire x1="121.92" y1="104.14" x2="121.92" y2="30.48" width="0.3048" layer="97" style="shortdash"/>
+<wire x1="121.92" y1="30.48" x2="121.92" y2="0" width="0.3048" layer="97" style="shortdash"/>
+<wire x1="0" y1="104.14" x2="86.36" y2="104.14" width="0.3048" layer="97" style="shortdash"/>
+<text x="127" y="180.34" size="2.54" layer="97">Shield Connections and controls</text>
+<wire x1="86.36" y1="104.14" x2="121.92" y2="104.14" width="0.3048" layer="97" style="shortdash"/>
+<wire x1="0" y1="30.48" x2="86.36" y2="30.48" width="0.3048" layer="97" style="shortdash"/>
+<text x="2.54" y="25.4" size="1.778" layer="97" align="top-left">MIDI I/O reference design from:
 http://www.midi.org/techspecs/electrispec.php
 JP1, JP2, JP3, JP4 implement power-over-MIDI, using pin assignment
@@
 Close JP1 &amp; 2 to power the MIDI input.
 Close JP3 &amp; 4 to power the output.</text>
-<text x="185.42" y="63.5" size="1.778" layer="94" align="top-left">Set S2 to "PROG" to load Sketch on
+<text x="185.42" y="63.5" size="1.778" layer="97" align="top-left">Set S2 to "PROG" to load Sketch on
 arduino, then set to "RUN" for MIDI
 communication
 LED1, LED2, RV1, RV2, S3, S4, and S5 are
 available for application usage.</text>
-<wire x1="86.36" y1="30.48" x2="121.92" y2="30.48" width="0.3048" layer="94" style="shortdash"/>
-<wire x1="86.36" y1="104.14" x2="86.36" y2="30.48" width="0.3048" layer="94" style="shortdash"/>
-<text x="88.9" y="96.52" size="2.54" layer="94">Serial Port
+<wire x1="86.36" y1="30.48" x2="121.92" y2="30.48" width="0.3048" layer="97" style="shortdash"/>
+<wire x1="86.36" y1="104.14" x2="86.36" y2="30.48" width="0.3048" layer="97" style="shortdash"/>
+<text x="88.9" y="96.52" size="2.54" layer="97">Serial Port
 Selection</text>
-<text x="88.9" y="50.8" size="1.778" layer="94" align="top-left">SJ1, SJ2 select
+<text x="88.9" y="50.8" size="1.778" layer="97" align="top-left">SJ1, SJ2 select
 between hardware
 serial port (pins 0, 1)
@@
 selected by default.
 </text>
+<text x="165.1" y="170.18" size="1.778" layer="97" align="top-left">Shield Vcc is provided by Arduino 5V line.
+The MIDI standard specifies 5V operation.</text>
 </plain>
 <instances>
@@
 <instance part="S1" gate="G$1" x="139.7" y="116.84"/>
 <instance part="S2" gate="1" x="220.98" y="142.24"/>
-<instance part="U$1" gate="G$1" x="76.2" y="160.02"/>
 <instance part="JP3" gate="G$1" x="48.26" y="55.88" smashed="yes" rot="R90">
 <attribute name="NAME" x="45.72" y="53.34" size="1.778" layer="95" rot="R90"/>
@@
 <instance part="SJ1" gate="G$1" x="101.6" y="83.82" rot="R180"/>
 <instance part="SJ2" gate="G$1" x="101.6" y="60.96" rot="R180"/>
+<instance part="U1" gate="G$1" x="76.2" y="160.02"/>
 </instances>
 <busses>
@@
 <wire x1="93.98" y1="152.4" x2="93.98" y2="147.32" width="0.1524" layer="91"/>
 <pinref part="GND1" gate="1" pin="GND"/>
-<pinref part="U$1" gate="G$1" pin="GND"/>
 <wire x1="88.9" y1="152.4" x2="93.98" y2="152.4" width="0.1524" layer="91"/>
+<pinref part="U1" gate="G$1" pin="GND"/>
 </segment>
 <segment>
@@
 <pinref part="P+1" gate="1" pin="VCC"/>
 <pinref part="R2" gate="G$1" pin="2"/>
-<pinref part="U$1" gate="G$1" pin="VCC"/>
 <wire x1="88.9" y1="162.56" x2="91.44" y2="162.56" width="0.1524" layer="91"/>
+<pinref part="U1" gate="G$1" pin="VCC"/>
 </segment>
 <segment>
@@
 <pinref part="D1" gate="G$1" pin="C"/>
 <pinref part="R1" gate="G$1" pin="2"/>
-<pinref part="U$1" gate="G$1" pin="A"/>
 <wire x1="66.04" y1="162.56" x2="63.5" y2="162.56" width="0.1524" layer="91"/>
 <junction x="63.5" y="162.56"/>
+<pinref part="U1" gate="G$1" pin="A"/>
 </segment>
 </net>
@@
 <wire x1="27.94" y1="134.62" x2="27.94" y2="152.4" width="0.1524" layer="91"/>
 <wire x1="27.94" y1="152.4" x2="63.5" y2="152.4" width="0.1524" layer="91"/>
-<pinref part="U$1" gate="G$1" pin="C"/>
 <wire x1="66.04" y1="152.4" x2="63.5" y2="152.4" width="0.1524" layer="91"/>
 <junction x="63.5" y="152.4"/>
+<pinref part="U1" gate="G$1" pin="C"/>
 </segment>
 </net>
@@
 <label x="106.68" y="157.48" size="1.27" layer="95" xref="yes"/>
 <pinref part="R2" gate="G$1" pin="1"/>
-<pinref part="U$1" gate="G$1" pin="VOUT"/>
 <wire x1="88.9" y1="157.48" x2="96.52" y2="157.48" width="0.1524" layer="91"/>
 <junction x="96.52" y="157.48"/>
-</segment>
-<segment>
+<pinref part="U1" gate="G$1" pin="VOUT"/>
+</segment>
+<segment>
