File: Hardware/SparkFun_MIDI_Shield.brd (EAGLE design)
At the start: 59.7 x 53.3 mm, 36 parts, among them J1 MIDI IN, J2 MIDI OUT, J3 UNO_R3_SHIELD, U1 6N138M, U2 74AHC1G125

Commit message: Fixing QC review issue with LP1,2 naming.
TX & RX were transposed in jumper names.
Parts:
- SJ1: value TX sel -> RX sel
- SJ2: value RX sel -> TX sel
Changed lines of the file:
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@@
 <setting verticaltext="up"/>
 </settings>
-<grid distance="0.01" unitdist="inch" unit="inch" style="lines" multiple="1" display="yes" altdistance="0.001" altunitdist="inch" altunit="inch"/>
+<grid distance="0.05" unitdist="inch" unit="inch" style="lines" multiple="1" display="yes" altdistance="0.005" altunitdist="inch" altunit="inch"/>
 <layers>
-<layer number="1" name="Top" color="4" fill="1" visible="yes" active="yes"/>
+<layer number="1" name="Top" color="4" fill="1" visible="no" active="yes"/>
 <layer number="2" name="Route2" color="1" fill="3" visible="no" active="no"/>
 <layer number="3" name="Route3" color="4" fill="3" visible="no" active="no"/>
@@
 <layer number="14" name="Route14" color="1" fill="6" visible="no" active="no"/>
 <layer number="15" name="Route15" color="4" fill="6" visible="no" active="no"/>
-<layer number="16" name="Bottom" color="1" fill="1" visible="yes" active="yes"/>
+<layer number="16" name="Bottom" color="1" fill="1" visible="no" active="yes"/>
 <layer number="17" name="Pads" color="2" fill="1" visible="yes" active="yes"/>
 <layer number="18" name="Vias" color="2" fill="1" visible="yes" active="yes"/>
@@
 <element name="LOGO3" library="SparkFun-Aesthetics" package="OSHW-LOGO-M" value="OSHW-LOGOM" x="38.1" y="26.67" rot="MR270"/>
 <element name="LOGO5" library="SparkFun-Aesthetics" package="SFE_LOGO_FLAME_.1" value="SFE_LOGO_FLAME.1_INCH" x="51.816" y="21.463" rot="R90"/>
-<element name="SJ1" library="SparkFun-Passives" package="PAD-JUMPER-3-2OF3_NC_BY_TRACE_YES_SILK_FULL_BOX" value="TX sel" x="25.4" y="45.72" rot="MR0"/>
-<element name="SJ2" library="SparkFun-Passives" package="PAD-JUMPER-3-2OF3_NC_BY_TRACE_YES_SILK_FULL_BOX" value="RX sel" x="19.05" y="45.72" rot="MR0"/>
+<element name="SJ1" library="SparkFun-Passives" package="PAD-JUMPER-3-2OF3_NC_BY_TRACE_YES_SILK_FULL_BOX" value="RX sel" x="25.4" y="45.72" rot="MR0"/>
+<element name="SJ2" library="SparkFun-Passives" package="PAD-JUMPER-3-2OF3_NC_BY_TRACE_YES_SILK_FULL_BOX" value="TX sel" x="19.05" y="45.72" rot="MR0"/>
 <element name="U1" library="SparkFun-DiscreteSemi" package="8-SMD" value="6N138M" x="25.4" y="29.21">
 <attribute name="PROD_ID" value="IC-09482" x="25.4" y="29.21" size="1.778" layer="27" font="vector" ratio="15" display="off"/>
